Commit message: left1

File: hb_task1b_ws/src/hb_task_1b/urdf/hb_bot.urdf.xacro (robot description, xacro)
@@ -107,4 +107,53 @@
         <material>Gazebo/Black</material>
     </gazebo>
+    <!-- left_wheel -->
+    <link name ="left_wheel">
+        <inertial>
+            <origin
+                xyz="0 -0.05 0.0"
+                rpy="1.57 0 0" />
+            <mass
+                value="0.060" />
+            <inertia
+                ixx="1.825e-4"
+                ixy="0"
+                ixz="0.00000000"
+                iyy="1.825e-4"
+                iyz="0"
+                izz="1.825e-4" />
+        </inertial>
+            <collision name="R_collision">
+            <origin
+                xyz="0 -0.05 0.0"
+                rpy="1.57 0 0" />
+            <geometry>
+            <cylinder length="0.13" radius="0.14"/>
+            </geometry>
+        </collision>
+        <visual>
+            <origin
+            xyz="0.0 0.0 0.0"
+            rpy="0.0 0.0 0.0" />
+            <geometry>
+                <mesh filename ="file://$(find holo)/meshes/wheel.stl" scale="5 5 5"/>
+            </geometry>
+        </visual>
+    </link>
+    <!-- Joint -->
+    <joint name ="left_wheel_joint" type="continuous" >
+        <origin
+                xyz="0.0 0.68 0.18"
+                rpy="0 0 0" />
+        <parent link="base_link"/>
+        <child link="left_wheel"/>
+        <axis xyz="0.0 1.0 0.0"/>
+         <limit
+            effort="5"
+            velocity="5" />
+    </joint>
+    <!-- material properties -->
+    <gazebo reference="left_wheel">
+        <material>Gazebo/Black</material>
+    </gazebo>
 <!-- ros_control plugin -->
   <gazebo>
