Commit message: bohoot kuch kiya

File: hb_task1b_ws/install/hb_task_1b/share/hb_task_1b/urdf/hb_bot.urdf.xacro (robot description, xacro)
@@ -105,5 +105,5 @@
     <!-- material properties -->
     <gazebo reference="right_wheel">
-        <material>Gazebo/Black</material>
+        <material>Gazebo/Blue</material>
     </gazebo>
     <!-- left_wheel -->
@@ -123,5 +123,5 @@
                 izz="1.825e-4" />
         </inertial>
-            <collision name="R_collision">
+            <collision name="l_collision">
             <origin
                 xyz="0 -0.05 0.0"
@@ -143,6 +143,6 @@
     <joint name ="left_wheel_joint" type="continuous" >
         <origin
-                xyz="0.0 0.68 0.18"
-                rpy="0 0 0" />
+                xyz="0.589 -0.34 0.18"
+                rpy="3.14 0 1.047" />
         <parent link="base_link"/>
         <child link="left_wheel"/>
@@ -154,4 +154,53 @@
     <!-- material properties -->
     <gazebo reference="left_wheel">
+        <material>Gazebo/red</material>
+    </gazebo>
+    <!-- rear_wheel -->
+    <link name ="rear_wheel">
+        <inertial>
+            <origin
+                xyz="0 -0.05 0.0"
+                rpy="1.57 0 0" />
+            <mass
+                value="0.060" />
+            <inertia
+                ixx="1.825e-4"
+                ixy="0"
+                ixz="0.00000000"
+                iyy="1.825e-4"
+                iyz="0"
+                izz="1.825e-4" />
+        </inertial>
+            <collision name="Re_collision">
+            <origin
+                xyz="0 -0.05 0.0"
+                rpy="1.57 0 0" />
+            <geometry>
+            <cylinder length="0.13" radius="0.14"/>
+            </geometry>
+        </collision>
+        <visual>
+            <origin
+            xyz="0.0 0.0 0.0"
+            rpy="0.0 0.0 0.0" />
+            <geometry>
+                <mesh filename ="/home/g10/eyrc_hb/hb_task1b_ws/src/hb_task_1b/meshes/wheel.stl" scale="5 5 5"/>
+            </geometry>
+        </visual>
+    </link>
+    <!-- Joint -->
+    <joint name ="rear_wheel_joint" type="continuous" >
+        <origin
+                xyz="-0.589 -0.34 0.18"
+                rpy="3.14 0 -1.047" />
+        <parent link="base_link"/>
+        <child link="rear_wheel"/>
+        <axis xyz="0.0 1.0 0.0"/>
+         <limit
+            effort="5"
+            velocity="5" />
+    </joint>
+    <!-- material properties -->
+    <gazebo reference="rear_wheel">
         <material>Gazebo/Black</material>
     </gazebo>

Commit message: bohoot kuch

File: hb_task1b_ws/install/hb_task_1b/share/hb_task_1b/urdf/hb_bot.urdf.xacro (robot description, xacro)
@@ -26,4 +26,7 @@
         <child link="base_link"/>
     </joint>
+    <gazebo reference="footprint_link">
+        <material>Gazebo/Black</material>
+    </gazebo>
     <!--Base link-->
     <link name ="base_link">
@@ -40,5 +43,5 @@
                 izz="0.011666666666667" />
         </inertial>
-         <collision name="collision">
+        <collision name="collision">
             <origin
                 xyz="0 0.0 0.28"
@@ -154,5 +157,5 @@
     <!-- material properties -->
     <gazebo reference="left_wheel">
-        <material>Gazebo/red</material>
+        <material>Gazebo/Red</material>
     </gazebo>
     <!-- rear_wheel -->
@@ -203,5 +206,5 @@
     <!-- material properties -->
     <gazebo reference="rear_wheel">
-        <material>Gazebo/Black</material>
+        <material>Gazebo/Green</material>
     </gazebo>
 <!-- ros_control plugin -->

File: hb_task1b_ws/src/hb_task_1b/urdf/hb_bot.urdf.xacro (robot description, xacro)
@@ -40,5 +40,5 @@
                 izz="0.011666666666667" />
         </inertial>
-         <collision name="collision">
+        <collision name="collision">
             <origin
                 xyz="0 0.0 0.28"
@@ -101,5 +101,5 @@
          <limit
             effort="5"
-            velocity="5000" />
+            velocity="5" />
     </joint>
     <!-- material properties -->
@@ -150,9 +150,9 @@
          <limit
             effort="5"
-            velocity="5000" />
+            velocity="5" />
     </joint>
     <!-- material properties -->
     <gazebo reference="left_wheel">
-        <material>Gazebo/red</material>
+        <material>Gazebo/Red</material>
     </gazebo>
     <!-- rear_wheel -->
@@ -199,9 +199,9 @@
          <limit
             effort="5"
-            velocity="5000" />
+            velocity="5" />
     </joint>
     <!-- material properties -->
     <gazebo reference="rear_wheel">
-        <material>Gazebo/Black</material>
+        <material>Gazebo/Green</material>
     </gazebo>
 <!-- ros_control plugin -->
